Commit message: Added batteries to weight down the robot

File: magni_description/urdf/magni.urdf.xacro (robot description, xacro)
@@ -3,5 +3,5 @@
   <xacro:arg name="raspicam_mount" default="forward"/>
   <xacro:property name="raspicam_mount" value="$(arg raspicam_mount)"/>
-  <xacro:arg name="sonars_installed" default="true"/>
+  <xacro:arg name="sonars_installed" default="false"/>
   <xacro:property name="sonars_installed" value="$(arg sonars_installed)"/>
   <xacro:arg name="camera_extrinsics_file" default="-"/>
@@ -9,7 +9,7 @@
   <xacro:arg name="lidar_installed" default="false"/>
   <xacro:property name="lidar_installed" value="$(arg lidar_installed)"/>
-  <xacro:arg name="velodyne_installed" default="false"/>
+  <xacro:arg name="velodyne_installed" default="true"/>
   <xacro:property name="velodyne_installed" value="$(arg velodyne_installed)"/>
-  <xacro:arg name="kinect_installed" default="true"/>
+  <xacro:arg name="kinect_installed" default="false"/>
   <xacro:property name="kinect_installed" value="$(arg kinect_installed)"/>
   <xacro:property name="wheel_r" value="0.1" />
@@ -22,7 +22,7 @@
   <xacro:include filename="$(find magni_description)/urdf/sensors/raspi_camera.xacro" />
   <xacro:include filename="$(find magni_description)/urdf/sensors/hokuyo_lidar.xacro" />
-  <xacro:include filename="$(find realsense2_description)/urdf/_d435.urdf.xacro" />
-  <xacro:include filename="$(find realsense2_description)/urdf/_d435.gazebo.xacro" />
-  <xacro:include filename="$(find turtlebot_description)/urdf/sensors/kinect.urdf.xacro" />
+  <!-- <xacro:include filename="$(find realsense2_description)/urdf/_d435.urdf.xacro" /> -->
+  <!-- <xacro:include filename="$(find realsense2_description)/urdf/_d435.gazebo.xacro" /> -->
+  <!-- <xacro:include filename="$(find turtlebot_description)/urdf/sensors/kinect.urdf.xacro" /> -->
   <!-- Robot base_link -->
   <link name="base_link">
@@ -79,4 +79,30 @@
     <child link="base_link"/>
     <origin xyz="0 0 ${wheel_r}" rpy="0 0 0"/>
+  </joint>
+  <!-- Place the batteries in the robot -->
+  <xacro:property name = "batt_width"  value = "${5.14*0.0254}"/>
+  <xacro:property name = "batt_length" value = "${7.72*0.0254}"/>
+  <xacro:property name = "batt_height" value = "${6.22*0.0254}"/>
+  <xacro:property name = "batt_mass"   value = "22.45"/>
+  <link name = "batteries">
+    <inertial name = "batteries_inertial">
+      <mass value = "${batt_mass}"/>
+      <inertia ixx = "${1/12.*batt_mass*(batt_length**2 + batt_height**2)}"
+               iyy = "${1/12.*batt_mass*(batt_width**2  + batt_height**2)}"
+               izz = "${1/12.*batt_mass*(batt_length**2 + batt_width**2)}"
+               ixy = "0" ixz = "0" iyz = "0"/>
+      <origin xyz = "0 0 ${batt_height/2}"/>
+    </inertial>
+    <!-- <visual name = "batteries_visual">
+      <origin xyz = "0 0 ${batt_height/2}"/>
+      <geometry>
+        <box size = "${2*batt_width} ${batt_length} ${batt_height}"/>
+      </geometry>
+    </visual> -->
+  </link>
+  <joint name = "battery_to_base_footprint" type = "fixed">
+    <parent link = "base_link"/>
+    <child  link = "batteries"/>
+    <origin  xyz = "-0.15 0 0"/>
   </joint>
   <!-- Macro for defining wheels -->
@@ -186,14 +212,14 @@
     </xacro:if>
   </xacro:if>
- <xacro:if value="${lidar_installed}">
+ <!-- <xacro:if value="${lidar_installed}">
     <xacro:hokuyo_lidar name="laser" connected_to="base_link">
       <origin xyz="0 0.0 0.2" rpy="0 0 0"/>
     </xacro:hokuyo_lidar>
-  </xacro:if>
-<xacro:if value="${kinect_installed}">
+  </xacro:if> -->
+<!-- <xacro:if value="${kinect_installed}">
     <xacro:sensor_d435  parent="base_link">
       <origin xyz="0.095 0.061 0.1" rpy="0 0 0"/>
     </xacro:sensor_d435>
-  </xacro:if>
+  </xacro:if> -->
  <xacro:if value="${velodyne_installed}">
 	<xacro:VLP-16 name="velodyne">

Commit message: Removed battery visual

File: magni_description/urdf/magni.urdf.xacro (robot description, xacro)
@@ -94,10 +94,4 @@
       <origin xyz = "0 0 ${batt_height/2}"/>
     </inertial>
-    <!-- <visual name = "batteries_visual">
-      <origin xyz = "0 0 ${batt_height/2}"/>
-      <geometry>
-        <box size = "${2*batt_width} ${batt_length} ${batt_height}"/>
-      </geometry>
-    </visual> -->
   </link>
   <joint name = "battery_to_base_footprint" type = "fixed">
@@ -212,14 +206,14 @@
     </xacro:if>
   </xacro:if>
- <!-- <xacro:if value="${lidar_installed}">
+ <xacro:if value="${lidar_installed}">
     <xacro:hokuyo_lidar name="laser" connected_to="base_link">
       <origin xyz="0 0.0 0.2" rpy="0 0 0"/>
     </xacro:hokuyo_lidar>
-  </xacro:if> -->
-<!-- <xacro:if value="${kinect_installed}">
+  </xacro:if>
+<xacro:if value="${kinect_installed}">
     <xacro:sensor_d435  parent="base_link">
       <origin xyz="0.095 0.061 0.1" rpy="0 0 0"/>
     </xacro:sensor_d435>
-  </xacro:if> -->
+  </xacro:if>
  <xacro:if value="${velodyne_installed}">
 	<xacro:VLP-16 name="velodyne">

Commit message: changed to built in inertia function

File: magni_description/urdf/magni.urdf.xacro (robot description, xacro)
@@ -86,17 +86,12 @@
   <xacro:property name = "batt_mass"   value = "22.45"/>
   <link name = "batteries">
-    <inertial name = "batteries_inertial">
-      <mass value = "${batt_mass}"/>
-      <inertia ixx = "${1/12.*batt_mass*(batt_length**2 + batt_height**2)}"
-               iyy = "${1/12.*batt_mass*(batt_width**2  + batt_height**2)}"
-               izz = "${1/12.*batt_mass*(batt_length**2 + batt_width**2)}"
-               ixy = "0" ixz = "0" iyz = "0"/>
-      <origin xyz = "0 0 ${batt_height/2}"/>
-    </inertial>
+    <xacro:box_inertial_with_origin x="${2*batt_width}" y="${batt_length}" z="${batt_height}" mass="${batt_mass}">
+      <origin xyz = "0 0 0" rpy = "0 0 0"/>
+    </xacro:box_inertial_with_origin>
   </link>
-  <joint name = "battery_to_base_footprint" type = "fixed">
+  <joint name = "battery_to_base_link" type = "continuous">
     <parent link = "base_link"/>
     <child  link = "batteries"/>
-    <origin  xyz = "-0.15 0 0"/>
+    <origin  xyz = "-0.15 0 ${batt_height/2}"/>
   </joint>
   <!-- Macro for defining wheels -->

Commit message: Made the urdf a little more readable

File: magni_description/urdf/magni.urdf.xacro (robot description, xacro)
@@ -33,5 +33,5 @@
       </geometry>
     </visual>
-	<visual>
+    <visual>
       <origin xyz="${-wheel_xpos-0.169} 0.17 ${-wheel_r+0.09}" rpy="0 0 ${pi}" />
       <geometry>
@@ -39,5 +39,5 @@
       </geometry>
     </visual>
-	<visual>
+    <visual>
       <origin xyz="${-wheel_xpos-0.169} -0.17 ${-wheel_r+0.09}" rpy="0 0 ${pi}" />
       <geometry>
@@ -46,5 +46,5 @@
     </visual>
     <collision>
-	  <origin xyz="${-wheel_xpos} 0 ${-wheel_r+0.151}" rpy="0 0 0" />
+      <origin xyz="${-wheel_xpos} 0 ${-wheel_r+0.151}" rpy="0 0 0" />
       <geometry>
         <box size="0.398 0.268 0.160"/>
@@ -201,17 +201,17 @@
     </xacro:if>
   </xacro:if>
- <xacro:if value="${lidar_installed}">
+  <xacro:if value="${lidar_installed}">
     <xacro:hokuyo_lidar name="laser" connected_to="base_link">
       <origin xyz="0 0.0 0.2" rpy="0 0 0"/>
     </xacro:hokuyo_lidar>
   </xacro:if>
-<xacro:if value="${kinect_installed}">
+  <xacro:if value="${kinect_installed}">
     <xacro:sensor_d435  parent="base_link">
       <origin xyz="0.095 0.061 0.1" rpy="0 0 0"/>
     </xacro:sensor_d435>
   </xacro:if>
- <xacro:if value="${velodyne_installed}">
-	<xacro:VLP-16 name="velodyne">
-      <origin xyz="0 0.0 0.3" rpy="0 0 0"/>
+  <xacro:if value="${velodyne_installed}">
+    <xacro:VLP-16 name="velodyne">
+        <origin xyz="0 0.0 0.3" rpy="0 0 0"/>
     </xacro:VLP-16>
   </xacro:if>

Commit message: fixed slight offset error of the back wheel

File: magni_description/urdf/magni.urdf.xacro (robot description, xacro)
@@ -87,5 +87,5 @@
     </xacro:box_inertial_with_origin>
   </link>
-  <joint name = "battery_to_base_link" type = "continuous">
+  <joint name = "battery_to_base_link" type = "fixed">
     <parent link = "base_link"/>
     <child  link = "batteries"/>
@@ -130,5 +130,5 @@
     <link name="${prefix}_caster_wheel">
       <collision>
-        <origin xyz="${-wheel_xpos-0.19} ${reflect*0.169} ${-wheel_r+0.04}" rpy="0 0 0" />
+        <origin xyz="${-wheel_xpos-0.19} ${reflect*0.169} ${-wheel_r+0.0435}" rpy="0 0 0" />
         <geometry>
           <sphere radius="0.04"/>

Commit message: Made base_link the parent of base_footprint

File: magni_description/urdf/magni.urdf.xacro (robot description, xacro)
@@ -73,7 +73,7 @@
   <link name="base_footprint"/>
   <joint name="base_footprint_joint" type="fixed">
-    <parent link="base_footprint"/>
-    <child link="base_link"/>
-    <origin xyz="0 0 ${wheel_r}" rpy="0 0 0"/>
+    <parent link="base_link"/>
+    <child link="base_footprint"/>
+    <origin xyz="0 0 ${-wheel_r}" rpy="0 0 0"/>
   </joint>
   <!-- Place the batteries in the robot -->

Commit message: fixed link order issue

File: magni_description/urdf/magni.urdf.xacro (robot description, xacro)
@@ -22,4 +22,6 @@
   <xacro:include filename="$(find magni_description)/urdf/sensors/raspi_camera.xacro" />
   <xacro:include filename="$(find magni_description)/urdf/sensors/hokuyo_lidar.xacro" />
+  <!-- First link -->
+  <link name="base_footprint"/>
   <!-- Robot base_link -->
   <link name="base_link">
@@ -71,9 +73,8 @@
   </link>
   <!-- Fixed offset from the floor to the center of the wheels -->
-  <link name="base_footprint"/>
   <joint name="base_footprint_joint" type="fixed">
-    <parent link="base_link"/>
-    <child link="base_footprint"/>
-    <origin xyz="0 0 ${-wheel_r}" rpy="0 0 0"/>
+    <parent link="base_footprint"/>
+    <child link="base_link"/>
+    <origin xyz="0 0 ${wheel_r}" rpy="0 0 0"/>
   </joint>
   <!-- Place the batteries in the robot -->
